File: AudioAmp.sch (KiCad schematic (older format))
At the start: 51 parts

Commit message: finished sch
Parts:
- added C1, C2: 47u, symbol Device:CP
- added C? (x3): 100n, symbol Device:C
- added C?: 220u, symbol Device:CP
- added D?: 1N4148, symbol Device:D_ALT
- added F? (x2): Fuse, symbol Device:Fuse
- added L?: L, symbol Device:L
- added Q?: 2SD600, Package_TO_SOT_THT:TO-126-3_Vertical, symbol Transistor_BJT:2SD600
- added Q?: 2SB631, Package_TO_SOT_THT:TO-126-3_Vertical, symbol Transistor_BJT:2SB631
- added Q?: 2SA1015, Package_TO_SOT_THT:TO-92_Inline, symbol Transistor_BJT:2SA1015
- added Q?: BC556, Package_TO_SOT_THT:TO-92_Inline, symbol Transistor_BJT:BC556
- added R? (x2): 100R, symbol Device:R
- added R? (x2): 270R, symbol Device:R
- added R? (x2): 0R22, symbol Device:R
- added R? (x2): 10R, symbol Device:R
- C?: value C -> 5p
- D? (x2): value D_ALT -> 1N4148
- R4: renamed from R?; value R -> 10K
- R? (x2): value R -> 68R
- R? (x2): value R -> 100R
- R? (x2): value R -> 330R
- R?: value R -> 10K
- gave numbers to parts that had none: 1
Connections:
- net labels added: IN, OUT, VCC, VSS
- wire segments 133 -> 192
Other:
- note added: "2N2219 -> 2N5551\n2N3905 -> 2N5401\n2SD600 -> 2SD669\nBC556 -> 2SA1302\n2SB631 -> 2SB649\n2SA1015 -> 2SC3281"
- note removed: "2N2219 -> 2N5551\n2N3905 -> 2N5401\n2SD600 -> 2SD669\n2SB631 -> 2SB649"

Commit message: set proper BJTs
Parts:
- removed Q? (x4): 2N3905, Package_TO_SOT_THT:TO-92_Inline, symbol Transistor_BJT:2N3905
- removed Q? (x3): 2SD600, Package_TO_SOT_THT:TO-126-3_Vertical, symbol Transistor_BJT:2SD600
- removed Q?: 2SB631, Package_TO_SOT_THT:TO-126-3_Vertical, symbol Transistor_BJT:2SB631
- added Q? (x4): 2N5401, Package_TO_SOT_THT:TO-92_Inline, symbol Pero_Kicad_Libraray:2N5401
- added Q?: 2SB649, Package_TO_SOT_THT:TO-92_Inline, symbol Pero_Kicad_Libraray:2SB649
- added Q? (x3): 2SD669, Package_TO_SOT_THT:TO-39-3, symbol Pero_Kicad_Libraray:2SD669
- L1: renamed from L?; value L -> 1u
- Q: renamed from Q?; value BC556 -> 2SA1302; symbol Transistor_BJT:BC556 -> Pero_Kicad_Libraray:2SA1302
- Q? (x4): value 2N2219 -> 2N5551; symbol Transistor_BJT:2N2219 -> Pero_Kicad_Libraray:2N5551
- Q?: value 2N3905 -> 2N5401; symbol Transistor_BJT:2N3905 -> Pero_Kicad_Libraray:2N5401
- Q?: value 2SB631 -> 2SB649; footprint Package_TO_SOT_THT:TO-126-3_Vertical -> Package_TO_SOT_THT:TO-92_Inline; symbol Transistor_BJT:2SB631 -> Pero_Kicad_Libraray:2SB649
- Q?: value 2SD600 -> 2SD669; footprint Package_TO_SOT_THT:TO-126-3_Vertical -> Package_TO_SOT_THT:TO-39-3; symbol Transistor_BJT:2SD600 -> Pero_Kicad_Libraray:2SD669
- Q?: value 2SA1015 -> 2SC3281; footprint Package_TO_SOT_THT:TO-92_Inline -> Package_TO_SOT_THT:TO-3PL; symbol Transistor_BJT:2SA1015 -> Pero_Kicad_Libraray:2SC3281
Connections:
- wire segments 192 -> 193
Other:
- note added: "Class B OPS with complimentary feedback"
- note added: "Complementary BJTs\n2N5551 - 2N5401, Ic = 0.6A, TO-92\n2SD669 - 2SB649, Ic = 1.5A, TO-126\n2SA1302 - 2SC3281, Ic = 15A, TO-3P"
- note added: "Current source for VA"
- note added: "Current source for diff. pair"
- note added: "Darlington VA stage with current limit"
- note added: "Input stage with current mirror and current source\n"
- note added: "OPS Bias"
- note added: "Single slope current limiter"
- note removed: "2N2219 -> 2N5551\n2N3905 -> 2N5401\n2SD600 -> 2SD669\nBC556 -> 2SA1302\n2SB631 -> 2SB649\n2SA1015 -> 2SC3281"

Commit message: found power resistors
Parts:
- removed R?: 0R22, symbol Device:R
- removed R?: 10R, symbol Device:R
- added R34: 0R22, Resistor_THT:R_Radial_Power_L13.0mm_W9.0mm_P5.00mm, symbol Pero_Kicad_Libraray:R
- added R36: 10R, Resistor_THT:R_Axial_DIN0516_L15.5mm_D5.0mm_P30.48mm_Horizontal, symbol Device:R
- D1, D2, D3: renamed from D?; footprint (none) -> Diode_THT:D_DO-34_SOD68_P10.16mm_Horizontal
- F1, F2: renamed from F?; footprint (none) -> Fuse:Fuseholder_Cylinder-5x20mm_Bulgin_FX0457_Horizontal_Closed
- Q10, Q11, Q14, Q8: renamed from Q?; footprint Package_TO_SOT_THT:TO-39-3 -> Package_TO_SOT_THT:TO-126-3_Horizontal_TabDown
- Q12, Q2, Q4, Q7: renamed from Q?; footprint Package_TO_SOT_THT:TO-39-3 -> Package_TO_SOT_THT:TO-92_Inline
- Q15, Q9: renamed from Q?; footprint Package_TO_SOT_THT:TO-92_Inline -> Package_TO_SOT_THT:TO-126-3_Horizontal_TabDown
- Q16: renamed from Q; footprint Package_TO_SOT_THT:TO-92_Inline -> Package_TO_SOT_THT:TO-3P-3_Vertical
- Q17: renamed from Q?; footprint Package_TO_SOT_THT:TO-3PL -> Package_TO_SOT_THT:TO-3P-3_Vertical
- R33: renamed from R?; footprint (none) -> Resistor_THT:R_Radial_Power_L13.0mm_W9.0mm_P5.00mm; symbol Device:R -> Pero_Kicad_Libraray:R; Manufacturer (none) -> TE Connectivty; Part Number (none) -> SQMW5R22J; RS Number (none) -> 199-7602; Resistance (none) -> 220 mΩ; Series (none) -> SQM5; Temp. coeff. (none) -> ±300ppm/°C; Tolerance (none) -> ±5%
- R35: renamed from R?; footprint (none) -> Resistor_THT:R_Axial_DIN0516_L15.5mm_D5.0mm_P30.48mm_Horizontal; Manufacturer (none) -> TE Connectivity; Part Number (none) -> CFR200J10R; RS Number (none) -> 131-621; Tolerance (none) -> ±5 %
- gave numbers to parts that had none: 47

Commit message: fixed BJT footprints, started placement
Parts:
- D1, D2, D3: footprint Diode_THT:D_DO-34_SOD68_P10.16mm_Horizontal -> (none)
- F1, F2: footprint Fuse:Fuseholder_Cylinder-5x20mm_Bulgin_FX0457_Horizontal_Closed -> (none)
- Q10, Q11, Q14, Q15, Q8, Q9: footprint Package_TO_SOT_THT:TO-126-3_Horizontal_TabDown -> Package_TO_SOT_THT:TO-126-3_Vertical
- R35, R36: footprint Resistor_THT:R_Axial_DIN0516_L15.5mm_D5.0mm_P30.48mm_Horizontal -> (none)
Changed lines of the file:
@@
 F 0 "Q9" H 5991 1896 50  0000 L CNN
 F 1 "2SB649" H 5991 1805 50  0000 L CNN
-F 2 "Package_TO_SOT_THT:TO-126-3_Horizontal_TabDown" H 6000 1775 50  0001 L CIN
+F 2 "Package_TO_SOT_THT:TO-126-3_Vertical" H 6000 1775 50  0001 L CIN
 F 3 "" H 5800 1850 50  0001 L CNN
 	1    5800 1850
@@
 F 0 "Q10" H 5991 3896 50  0000 L CNN
 F 1 "2SD669" H 5991 3805 50  0000 L CNN
-F 2 "Package_TO_SOT_THT:TO-126-3_Horizontal_TabDown" H 6000 3775 50  0001 L CIN
+F 2 "Package_TO_SOT_THT:TO-126-3_Vertical" H 6000 3775 50  0001 L CIN
 F 3 "" H 5800 3850 50  0001 L CNN
 	1    5800 3850
@@
 F 0 "D2" V 6596 2971 50  0000 R CNN
 F 1 "1N4148" V 6505 2971 50  0000 R CNN
-F 2 "Diode_THT:D_DO-34_SOD68_P10.16mm_Horizontal" H 6550 3050 50  0001 C CNN
+F 2 "" H 6550 3050 50  0001 C CNN
 F 3 "" H 6550 3050 50  0001 C CNN
 	1    6550 3050
@@
 F 0 "D3" V 6596 4571 50  0000 R CNN
 F 1 "1N4148" V 6505 4571 50  0000 R CNN
-F 2 "Diode_THT:D_DO-34_SOD68_P10.16mm_Horizontal" H 6550 4650 50  0001 C CNN
+F 2 "" H 6550 4650 50  0001 C CNN
 F 3 "" H 6550 4650 50  0001 C CNN
 	1    6550 4650
@@
 F 0 "D1" V 4154 4479 50  0000 L CNN
 F 1 "1N4148" V 4245 4479 50  0000 L CNN
-F 2 "Diode_THT:D_DO-34_SOD68_P10.16mm_Horizontal" H 4200 4400 50  0001 C CNN
+F 2 "" H 4200 4400 50  0001 C CNN
 F 3 "" H 4200 4400 50  0001 C CNN
 	1    4200 4400
@@
 F 0 "R35" H 9320 4141 50  0000 L CNN
 F 1 "10R" H 9320 4050 50  0000 L CNN
-F 2 "Resistor_THT:R_Axial_DIN0516_L15.5mm_D5.0mm_P30.48mm_Horizontal" V 9180 4050 50  0001 C CNN
+F 2 "" V 9180 4050 50  0001 C CNN
 F 3 "https://at.rs-online.com/web/p/products/0131621/" H 9250 4050 50  0001 C CNN
 F 4 "2W" H 9320 3959 50  0000 L CNN "Power"
@@
 F 0 "F1" V 9503 6150 50  0000 C CNN
 F 1 "Fuse" V 9594 6150 50  0000 C CNN
-F 2 "Fuse:Fuseholder_Cylinder-5x20mm_Bulgin_FX0457_Horizontal_Closed" V 9630 6150 50  0001 C CNN
+F 2 "" V 9630 6150 50  0001 C CNN
 F 3 "" H 9700 6150 50  0001 C CNN
 	1    9700 6150
@@
 F 0 "F2" V 9553 1100 50  0000 C CNN
 F 1 "Fuse" V 9644 1100 50  0000 C CNN
-F 2 "Fuse:Fuseholder_Cylinder-5x20mm_Bulgin_FX0457_Horizontal_Closed" V 9680 1100 50  0001 C CNN
+F 2 "" V 9680 1100 50  0001 C CNN
 F 3 "" H 9750 1100 50  0001 C CNN
 	1    9750 1100
@@
 F 0 "Q15" H 8100 4820 50  0000 L CNN
 F 1 "2SB649" H 8100 4900 50  0000 L CNN
-F 2 "Package_TO_SOT_THT:TO-126-3_Horizontal_TabDown" H 8100 4775 50  0001 L CIN
+F 2 "Package_TO_SOT_THT:TO-126-3_Vertical" H 8100 4775 50  0001 L CIN
 F 3 "" H 7900 4850 50  0001 L CNN
 	1    7900 4850
@@
 F 0 "Q14" H 8091 2896 50  0000 L CNN
 F 1 "2SD669" H 8091 2805 50  0000 L CNN
-F 2 "Package_TO_SOT_THT:TO-126-3_Horizontal_TabDown" H 8100 2775 50  0001 L CIN
+F 2 "Package_TO_SOT_THT:TO-126-3_Vertical" H 8100 2775 50  0001 L CIN
 F 3 "" H 7900 2850 50  0001 L CNN
 	1    7900 2850
@@
 F 0 "Q11" H 5991 5596 50  0000 L CNN
 F 1 "2SD669" H 5991 5505 50  0000 L CNN
-F 2 "Package_TO_SOT_THT:TO-126-3_Horizontal_TabDown" H 6000 5475 50  0001 L CIN
+F 2 "Package_TO_SOT_THT:TO-126-3_Vertical" H 6000 5475 50  0001 L CIN
 F 3 "" H 5800 5550 50  0001 L CNN
 	1    5800 5550
@@
 F 0 "Q8" H 5541 5396 50  0000 L CNN
 F 1 "2SD669" H 5541 5305 50  0000 L CNN
-F 2 "Package_TO_SOT_THT:TO-126-3_Horizontal_TabDown" H 5550 5275 50  0001 L CIN
+F 2 "Package_TO_SOT_THT:TO-126-3_Vertical" H 5550 5275 50  0001 L CIN
 F 3 "" H 5350 5350 50  0001 L CNN
 	1    5350 5350
@@
 F 0 "R36" V 9710 3790 50  0000 L CNN
 F 1 "10R" V 9800 3790 50  0000 L CNN
-F 2 "Resistor_THT:R_Axial_DIN0516_L15.5mm_D5.0mm_P30.48mm_Horizontal" V 9530 3850 50  0001 C CNN
+F 2 "" V 9530 3850 50  0001 C CNN
 F 3 "https://at.rs-online.com/web/p/products/0131621/" H 9600 3850 50  0001 C CNN
 F 4 "2W" V 9890 3790 50  0000 L CNN "Power"

Commit message: connectors and fuses added
Parts:
- added J1, J2, J3, J4, J5: Conn_01x01, Connectors:Pin_d0.7mm_L6.5mm_W1.8mm_FlatFork, symbol Connector_Generic:Conn_01x01
- F1, F2: footprint (none) -> Fuse_Holders_and_Fuses:Fuseholder5x20_horiz_open_inline_Type-I; RS Number (none) -> 769-0168
Connections:
- wire segments 193 -> 201

Commit message: placement done
Parts:
- C1, C2, C5, C6: footprint (none) -> Capacitors_THT:CP_Radial_D10.0mm_P5.00mm
- C11, C12, C13: footprint (none) -> Capacitors_THT:C_Rect_L10.0mm_W4.0mm_P7.50mm_MKS4
- C3, C4: footprint (none) -> Capacitors_THT:CP_Radial_D22.0mm_P10.00mm_SnapIn
- C7, C9: footprint (none) -> Capacitors_THT:C_Rect_L10.0mm_W3.0mm_P7.50mm_MKS4
- C8: footprint (none) -> Capacitors_THT:C_Disc_D6.0mm_W2.5mm_P5.00mm
- F1, F2: Rating (none) -> 2A
- R1, R10, R11, R12, R13, R14, R15, R16, R17, R18, R19, R2, R20, R21, R22, R23, R24, R25, R26, R27, R28, R29, R3, R30, R31, R32, R4, R5, R6, R7, R8, R9: footprint (none) -> Resistors_THT:R_Axial_DIN0207_L6.3mm_D2.5mm_P10.16mm_Horizontal
- R35, R36: footprint (none) -> Resistors_THT:R_Axial_DIN0516_L15.5mm_D5.0mm_P30.48mm_Horizontal
- RV1: footprint (none) -> Potentiometers:Potentiometer_Trimmer_Piher_PT-10v10_Horizontal_Px10.0mm_Py5.0mm
Connections:
- net labels added: VCC_FUSED, VSS_FUSED

Commit message: routed
Parts:
- J3, J4, J5: footprint Connectors:Pin_d0.7mm_L6.5mm_W1.8mm_FlatFork -> Flachsteceker:216843-1
Changed lines of the file:
@@
 F 0 "J4" H 10780 6146 50  0000 L CNN
 F 1 "Conn_01x01" H 10780 6101 50  0001 L CNN
-F 2 "Connectors:Pin_d0.7mm_L6.5mm_W1.8mm_FlatFork" H 10700 6150 50  0001 C CNN
+F 2 "Flachsteceker:216843-1" H 10700 6150 50  0001 C CNN
 F 3 "~" H 10700 6150 50  0001 C CNN
 	1    10700 6150
@@
 F 0 "J5" H 10780 1596 50  0000 L CNN
 F 1 "Conn_01x01" H 10780 1551 50  0001 L CNN
-F 2 "Connectors:Pin_d0.7mm_L6.5mm_W1.8mm_FlatFork" H 10700 1600 50  0001 C CNN
+F 2 "Flachsteceker:216843-1" H 10700 1600 50  0001 C CNN
 F 3 "~" H 10700 1600 50  0001 C CNN
 	1    10700 1600
@@
 F 0 "J3" H 10779 1096 50  0000 L CNN
 F 1 "Conn_01x01" H 10780 1051 50  0001 L CNN
-F 2 "Connectors:Pin_d0.7mm_L6.5mm_W1.8mm_FlatFork" H 10700 1100 50  0001 C CNN
+F 2 "Flachsteceker:216843-1" H 10700 1100 50  0001 C CNN
 F 3 "~" H 10700 1100 50  0001 C CNN
 	1    10700 1100
