File: AudioAmp.sch (KiCad schematic (older format))
At the start: 78 parts, among them J1 Conn_01x01, J2 Conn_01x01, J3 Conn_01x01, J4 Conn_01x01, J5 Conn_01x01, Q1 2N5401, Q10 2SD669, Q11 2SD669, Q12 2N5551, Q13 2N5401, Q14 2SD669, Q15 2SB649, Q16 2SA1302, Q17 2SC3281, Q2 2N5551, Q3 2N5401, Q4 2N5551, Q5 2N5401, Q6 2N5401, Q7 2N5551, Q8 2SD669, Q9 2SB649

Commit message: silkscreen
Parts:
- F1, F2: Rating 2A -> 3A
Other:
- note added: "Ic=6.5mA"
- note added: "Ilim = .65/.22 = 3A"
Changed lines of the file:
@@
 F 3 "" H 10000 1100 50  0001 C CNN
 F 4 " 769-0168" V 10200 1100 50  0000 C CNN "RS Number"
-F 5 "2A" V 10100 1100 50  0000 C CNN "Rating"
+F 5 "3A" V 10100 1100 50  0000 C CNN "Rating"
 	1    10000 1100
 	0    1    1    0
@@
 F 3 "" H 9950 6150 50  0001 C CNN
 F 4 " 769-0168" V 10150 6150 50  0000 C CNN "RS Number"
-F 5 "2A" V 10050 6150 50  0000 C CNN "Rating"
+F 5 "3A" V 10050 6150 50  0000 C CNN "Rating"
 	1    9950 6150
 	0    1    1    0
@@
 Text Label 8950 6150 0    50   ~ 0
 VSS_FUSED
+Text Notes 7910 3720 0    50   ~ 0
+Ilim = .65/.22 = 3A
+Text Notes 6500 1340 0    50   ~ 0
+Ic=6.5mA
 $EndSCHEMATC

Commit message: in/out connectors, silkscreen check
Parts:
- added J6, J7, J8: Conn_01x01, Flachsteceker:216843-1, symbol Connector_Generic:Conn_01x01
- J1, J2: footprint Connectors:Pin_d0.7mm_L6.5mm_W1.8mm_FlatFork -> Flachsteceker:216843-1
Connections:
- net GND: now also J6.1 (Pin_1), J7.1 (Pin_1), J8.1 (Pin_1)
Changed lines of the file:
@@
 F 0 "J2" H 10479 4096 50  0000 L CNN
 F 1 "Conn_01x01" H 10480 4051 50  0001 L CNN
-F 2 "Connectors:Pin_d0.7mm_L6.5mm_W1.8mm_FlatFork" H 10400 4100 50  0001 C CNN
+F 2 "Flachsteceker:216843-1" H 10400 4100 50  0001 C CNN
 F 3 "~" H 10400 4100 50  0001 C CNN
 	1    10400 4100
@@
 F 0 "J1" H 820 3467 50  0000 C CNN
 F 1 "Conn_01x01" H 980 3551 50  0001 L CNN
-F 2 "Connectors:Pin_d0.7mm_L6.5mm_W1.8mm_FlatFork" H 900 3600 50  0001 C CNN
+F 2 "Flachsteceker:216843-1" H 900 3600 50  0001 C CNN
 F 3 "~" H 900 3600 50  0001 C CNN
 	1    900  3600
@@
 Text Notes 6500 1340 0    50   ~ 0
 Ic=6.5mA
+$Comp
+L Connector_Generic:Conn_01x01 J6
+U 1 1 5C462001
+P 900 4200
+F 0 "J6" H 820 4067 50  0000 C CNN
+F 1 "Conn_01x01" H 980 4151 50  0001 L CNN
+F 2 "Flachsteceker:216843-1" H 900 4200 50  0001 C CNN
+F 3 "~" H 900 4200 50  0001 C CNN
+	1    900  4200
+	-1   0    0    1
+$EndComp
+$Comp
+L power:GND #PWR012
+U 1 1 5C4621BC
+P 1100 4350
+F 0 "#PWR012" H 1100 4100 50  0001 C CNN
+F 1 "GND" H 1105 4177 50  0000 C CNN
+F 2 "" H 1100 4350 50  0001 C CNN
+F 3 "" H 1100 4350 50  0001 C CNN
+	1    1100 4350
+	1    0    0    -1
+$EndComp
+Wire Wire Line
+	1100 4200 1100 4350
+$Comp
+L Connector_Generic:Conn_01x01 J7
+U 1 1 5C48829D
+P 10400 4550
+F 0 "J7" H 10479 4546 50  0000 L CNN
+F 1 "Conn_01x01" H 10480 4501 50  0001 L CNN
+F 2 "Flachsteceker:216843-1" H 10400 4550 50  0001 C CNN
+F 3 "~" H 10400 4550 50  0001 C CNN
+	1    10400 4550
+	1    0    0    -1
+$EndComp
+$Comp
+L power:GND #PWR013
+U 1 1 5C4883A9
+P 10150 4750
+F 0 "#PWR013" H 10150 4500 50  0001 C CNN
+F 1 "GND" H 10155 4577 50  0000 C CNN
+F 2 "" H 10150 4750 50  0001 C CNN
+F 3 "" H 10150 4750 50  0001 C CNN
+	1    10150 4750
+	1    0    0    -1
+$EndComp
+Wire Wire Line
+	10150 4750 10150 4550
+Wire Wire Line
+	10150 4550 10200 4550
+$Comp
+L Connector_Generic:Conn_01x01 J8
+U 1 1 5C492DC1
+P 10700 5750
+F 0 "J8" H 10780 5746 50  0000 L CNN
+F 1 "Conn_01x01" H 10780 5701 50  0001 L CNN
+F 2 "Flachsteceker:216843-1" H 10700 5750 50  0001 C CNN
+F 3 "~" H 10700 5750 50  0001 C CNN
+	1    10700 5750
+	1    0    0    -1
+$EndComp
+$Comp
+L power:GND #PWR0101
+U 1 1 5C4933A6
+P 10400 5850
+F 0 "#PWR0101" H 10400 5600 50  0001 C CNN
+F 1 "GND" H 10405 5677 50  0000 C CNN
+F 2 "" H 10400 5850 50  0001 C CNN
+F 3 "" H 10400 5850 50  0001 C CNN
+	1    10400 5850
+	1    0    0    -1
+$EndComp
+Wire Wire Line
+	10400 5850 10400 5750
+Wire Wire Line
+	10400 5750 10500 5750
 $EndSCHEMATC

Commit message: fixed Q9 and simulation
Connections:
- net at R14.1, R20.2: now also Q9.1 (E); no longer Q9.2 (C)
- net at C10.1, R18.1, R21.1: now also Q9.2 (C); no longer Q9.1 (E)
Other:
- note added: "Ilim = .65/.3/.22 = 9.8A"
- note removed: "Ilim = .65/.22 = 3A"
Changed lines of the file:
@@
 F 3 "" H 6050 1850 50  0001 L CNN
 	1    6050 1850
-	1    0    0    -1
+	1    0    0    1
 $EndComp
 Wire Wire Line
@@
 Text Label 8950 6150 0    50   ~ 0
 VSS_FUSED
-Text Notes 7910 3720 0    50   ~ 0
-Ilim = .65/.22 = 3A
+Text Notes 7850 3700 0    50   ~ 0
+Ilim = .65/.3/.22 = 9.8A
 Text Notes 6500 1340 0    50   ~ 0
 Ic=6.5mA

Commit message: fixed libraries, now works everything, including 3d models
Parts:
- C1, C2, C5, C6: footprint Capacitors_THT:CP_Radial_D10.0mm_P5.00mm -> Capacitor_THT:CP_Radial_D10.0mm_P5.00mm
- C11, C12, C13: footprint Capacitors_THT:C_Rect_L10.0mm_W4.0mm_P7.50mm_MKS4 -> Capacitor_THT:C_Rect_L10.0mm_W4.0mm_P7.50mm_MKS4
- C3, C4: footprint Capacitors_THT:CP_Radial_D22.0mm_P10.00mm_SnapIn -> Capacitor_THT:CP_Radial_D22.0mm_P10.00mm_SnapIn
- C7, C9: footprint Capacitors_THT:C_Rect_L10.0mm_W3.0mm_P7.50mm_MKS4 -> Capacitor_THT:C_Rect_L10.0mm_W3.0mm_P7.50mm_MKS4
- C8: footprint Capacitors_THT:C_Disc_D6.0mm_W2.5mm_P5.00mm -> Capacitor_THT:C_Disc_D6.0mm_W2.5mm_P5.00mm
- F1, F2: footprint Fuse_Holders_and_Fuses:Fuseholder5x20_horiz_open_inline_Type-I -> Fuse:Fuseholder_Cylinder-5x20mm_Schurter_0031_8201_Horizontal_Open
- R1, R10, R11, R12, R13, R14, R15, R16, R17, R18, R19, R2, R20, R21, R22, R23, R24, R25, R26, R27, R28, R29, R3, R30, R31, R32, R4, R5, R6, R7, R8, R9: footprint Resistors_THT:R_Axial_DIN0207_L6.3mm_D2.5mm_P10.16mm_Horizontal -> Resistor_THT:R_Axial_DIN0207_L6.3mm_D2.5mm_P10.16mm_Horizontal
- R35, R36: footprint Resistors_THT:R_Axial_DIN0516_L15.5mm_D5.0mm_P30.48mm_Horizontal -> Resistor_THT:R_Axial_DIN0516_L15.5mm_D5.0mm_P30.48mm_Horizontal
- RV1: footprint Potentiometers:Potentiometer_Trimmer_Piher_PT-10v10_Horizontal_Px10.0mm_Py5.0mm -> Potentiometer_THT:Potentiometer_Piher_PT-10-V10_Vertical
