File: AudioAmp.kicad_pcb (KiCad board)
At the start: 2 copper layers, 62 parts, among them Q1 2N5401, Q10 2SD669, Q11 2SD669, Q12 2N5551, Q13 2N5401, Q14 2SD669, Q15 2SB649, Q16 2SA1302, Q17 2SC3281, Q2 2N5551, Q3 2N5401, Q4 2N5551, Q5 2N5401, Q6 2N5401, Q7 2N5551, Q8 2SD669, Q9 2SB649

Commit message: preliminary placement, caps missing
Parts:
- moved L1 179.2 mm to (165.0, 145.0), turned to 90 degrees
- moved R35 144.5 mm to (170.0, 72.0), turned to 270 degrees
- moved R36 113.3 mm to (157.5, 102.5), turned to 90 degrees
- moved C13 105.8 mm to (152.5, 145.0), turned to 90 degrees
- moved R13 105.0 mm to (102.5, 130.0), turned to 270 degrees
- moved R32 103.6 mm to (145.0, 130.0), turned to 270 degrees
- moved R34 100.9 mm to (145.0, 120.0), turned to 90 degrees
- moved Q8 92.9 mm to (112.5, 124.3), turned to 90 degrees
- moved D3 88.0 mm to (122.5, 140.2), turned to 90 degrees
- moved R28 87.2 mm to (130.0, 130.0), turned to 270 degrees
- moved R30 86.4 mm to (135.0, 112.5), turned to 270 degrees
- moved Q11 83.2 mm to (117.5, 124.3), turned to 90 degrees
- moved R17 82.7 mm to (107.5, 130.0), turned to 270 degrees
- moved R31 80.0 mm to (145.0, 90.0), turned to 90 degrees
- moved R23 79.8 mm to (117.5, 140.2), turned to 90 degrees
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Other:
- board outline added: 130 x 85 mm

Commit message: connectors and fuses added
Parts:
- added J1: Conn_01x01, Connectors:Pin_d0.7mm_L6.5mm_W1.8mm_FlatFork, F.Cu at (62.0, 94.2)
- added J2: Conn_01x01, Connectors:Pin_d0.7mm_L6.5mm_W1.8mm_FlatFork, F.Cu at (154.7, 106.7)
- added J3: Conn_01x01, Connectors:Pin_d0.7mm_L6.5mm_W1.8mm_FlatFork, F.Cu at (117.6, 73.7)
- added J4: Conn_01x01, Connectors:Pin_d0.7mm_L6.5mm_W1.8mm_FlatFork, F.Cu at (116.6, 145.5)
- added J5: Conn_01x01, Connectors:Pin_d0.7mm_L6.5mm_W1.8mm_FlatFork, F.Cu at (175.0, 71.9)
- F1, F2: footprint Fuse:Fuseholder_Cylinder-5x20mm_Bulgin_FX0457_Horizontal_Closed -> Fuse_Holders_and_Fuses:Fuseholder5x20_horiz_open_inline_Type-I
- moved F1 139.0 mm to (123.7, 145.5)
- moved F2 107.1 mm to (125.5, 73.7)
Connections:
- F1 pad 1: (no net) -> VSS
- F2 pad 1: (no net) -> VCC
- R12 pad 1: (no net) -> Net-(C8-Pad2)
- R13 pad 1: (no net) -> Net-(C7-Pad1)
- R19 pad 2: (no net) -> Net-(R19-Pad2)

Commit message: placement done
Parts:
- added C1: 47u, Capacitors_THT:CP_Radial_D10.0mm_P5.00mm, F.Cu at (95.5, 66.7)
- added C2: 47u, Capacitors_THT:CP_Radial_D10.0mm_P5.00mm, F.Cu at (95.5, 89.0)
- added C3: 220u, Capacitors_THT:CP_Radial_D22.0mm_P10.00mm_SnapIn, F.Cu at (203.0, 123.7)
- added C4: 220u, Capacitors_THT:CP_Radial_D22.0mm_P10.00mm_SnapIn, F.Cu at (203.0, 66.3)
- added C5: 47u, Capacitors_THT:CP_Radial_D10.0mm_P5.00mm, F.Cu at (107.5, 66.7)
- added C6: 220u, Capacitors_THT:CP_Radial_D10.0mm_P5.00mm, F.Cu at (122.0, 121.0)
- added C7: 150p, Capacitors_THT:C_Rect_L10.0mm_W3.0mm_P7.50mm_MKS4, F.Cu at (129.0, 126.7)
- added C8: 5p, Capacitors_THT:C_Disc_D6.0mm_W2.5mm_P5.00mm, F.Cu at (154.6, 89.0)
- added C9: 300p, Capacitors_THT:C_Rect_L10.0mm_W3.0mm_P7.50mm_MKS4, F.Cu at (138.0, 113.0)
- added RV1: 1K, Potentiometers:Potentiometer_Trimmer_Piher_PT-10v10_Horizontal_Px10.0mm_Py5.0mm, F.Cu at (152.7, 97.0)
- C11, C12, C13: footprint Capacitor_THT:C_Rect_L7.0mm_W4.5mm_P5.00mm -> Capacitors_THT:C_Rect_L10.0mm_W4.0mm_P7.50mm_MKS4
- R1, R10, R11, R12, R13, R14, R15, R16, R17, R18, R19, R2, R20, R21, R22, R23, R24, R25, R26, R27, R28, R29, R3, R30, R31, R32, R4, R5, R6, R7, R8, R9: footprint Resistor_THT:R_Axial_DIN0207_L6.3mm_D2.5mm_P10.16mm_Horizontal -> Resistors_THT:R_Axial_DIN0207_L6.3mm_D2.5mm_P10.16mm_Horizontal
- R35, R36: footprint Resistor_THT:R_Axial_DIN0516_L15.5mm_D5.0mm_P30.48mm_Horizontal -> Resistors_THT:R_Axial_DIN0516_L15.5mm_D5.0mm_P30.48mm_Horizontal
- moved L1 74.8 mm to (194.0, 76.0), turned to 270 degrees
- moved C13 67.5 mm to (219.0, 133.2)
- moved C11 57.6 mm to (219.0, 56.9), turned to 270 degrees
- moved Q16 54.1 mm to (225.5, 52.5)
- moved Q14 52.4 mm to (227.0, 75.8)
- moved Q10 50.5 mm to (227.0, 92.5)
- moved R36 49.7 mm to (207.0, 107.2)
- moved Q15 49.2 mm to (227.0, 109.1)
- moved J1 48.3 mm to (95.5, 59.5)
- moved Q17 47.9 mm to (226.0, 126.6)
- moved R35 46.2 mm to (216.0, 76.7)
- moved C12 44.1 mm to (208.0, 112.5), turned to 0 degrees
- moved J3 43.2 mm to (154.5, 51.1)
- moved F2 42.1 mm to (162.5, 53.6)
- moved R24 40.7 mm to (154.6, 63.1)
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Connections:
- net Net-(C11-Pad2) renamed /VCC_FUSED
- net Net-(C13-Pad1) renamed /VSS_FUSED
Other:
- board size 130 x 85 mm -> 160 x 100 mm
- net class HIGH_CURRENT added: clearance 0.5, trace_width 1, via_dia 0.8, via_drill 0.4

Commit message: mounting holes
Parts:
- added REF**: MountingHole_3.5mm, Mounting_Holes:MountingHole_3.5mm, F.Cu at (219.0, 139.0)
- added REF**: MountingHole_3.5mm, Mounting_Holes:MountingHole_3.5mm, F.Cu at (219.0, 50.0)
- added REF**: MountingHole_3.5mm, Mounting_Holes:MountingHole_3.5mm, F.Cu at (80.0, 135.0)
- added REF**: MountingHole_3.5mm, Mounting_Holes:MountingHole_3.5mm, F.Cu at (80.0, 55.0)
Routing:
- net (no net): vias 0 -> 1
Changed lines of the file:
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@@
     (thickness 1.6)
     (drawings 10)
-    (tracks 0)
+    (tracks 1)
     (zones 0)
-    (modules 77)
+    (modules 81)
     (nets 48)
   )
@@
     (add_net VSS)
   )
+  (module Mounting_Holes:MountingHole_3.5mm (layer F.Cu)
+    (at 219 139)
+    (descr "Mounting Hole 3.5mm, no annular")
+    (tags "mounting hole 3.5mm no annular")
+    (attr virtual)
+    (fp_text reference REF** (at 0 -4.5) (layer F.SilkS)
+      (effects (font (size 1 1) (thickness 0.15)))
+    )
+    (fp_text value MountingHole_3.5mm (at 0 4.5) (layer F.Fab)
+      (effects (font (size 1 1) (thickness 0.15)))
+    )
+    (fp_text user %R (at 0.3 0) (layer F.Fab)
+      (effects (font (size 1 1) (thickness 0.15)))
+    )
+    (fp_circle (center 0 0) (end 3.5 0) (layer Cmts.User) (width 0.15))
+    (fp_circle (center 0 0) (end 3.75 0) (layer F.CrtYd) (width 0.05))
+    (pad 1 np_thru_hole circle (at 0 0) (size 3.5 3.5) (drill 3.5) (layers *.Cu *.Mask))
+  )
+  (module Mounting_Holes:MountingHole_3.5mm (layer F.Cu)
+    (at 219 50)
+    (descr "Mounting Hole 3.5mm, no annular")
+    (tags "mounting hole 3.5mm no annular")
+    (attr virtual)
+    (fp_text reference REF** (at 0 -4.5) (layer F.SilkS)
+      (effects (font (size 1 1) (thickness 0.15)))
+    )
+    (fp_text value MountingHole_3.5mm (at 0 4.5) (layer F.Fab)
+      (effects (font (size 1 1) (thickness 0.15)))
+    )
+    (fp_text user %R (at 0.3 0) (layer F.Fab)
+      (effects (font (size 1 1) (thickness 0.15)))
+    )
+    (fp_circle (center 0 0) (end 3.5 0) (layer Cmts.User) (width 0.15))
+    (fp_circle (center 0 0) (end 3.75 0) (layer F.CrtYd) (width 0.05))
+    (pad 1 np_thru_hole circle (at 0 0) (size 3.5 3.5) (drill 3.5) (layers *.Cu *.Mask))
+  )
+  (module Mounting_Holes:MountingHole_3.5mm (layer F.Cu)
+    (at 80 135)
+    (descr "Mounting Hole 3.5mm, no annular")
+    (tags "mounting hole 3.5mm no annular")
+    (attr virtual)
+    (fp_text reference REF** (at 0 -4.5) (layer F.SilkS)
+      (effects (font (size 1 1) (thickness 0.15)))
+    )
+    (fp_text value MountingHole_3.5mm (at 0 4.5) (layer F.Fab)
+      (effects (font (size 1 1) (thickness 0.15)))
+    )
+    (fp_text user %R (at 0.3 0) (layer F.Fab)
+      (effects (font (size 1 1) (thickness 0.15)))
+    )
+    (fp_circle (center 0 0) (end 3.5 0) (layer Cmts.User) (width 0.15))
+    (fp_circle (center 0 0) (end 3.75 0) (layer F.CrtYd) (width 0.05))
+    (pad 1 np_thru_hole circle (at 0 0) (size 3.5 3.5) (drill 3.5) (layers *.Cu *.Mask))
+  )
   (module Connectors:Pin_d0.7mm_L6.5mm_W1.8mm_FlatFork (layer F.Cu)
     (at 154.5 51.15)
@@
     )
   )
+  (module Mounting_Holes:MountingHole_3.5mm (layer F.Cu)
+    (at 80 55)
+    (descr "Mounting Hole 3.5mm, no annular")
+    (tags "mounting hole 3.5mm no annular")
+    (attr virtual)
+    (fp_text reference REF** (at 0 -4.5) (layer F.SilkS)
+      (effects (font (size 1 1) (thickness 0.15)))
+    )
+    (fp_text value MountingHole_3.5mm (at 0 4.5) (layer F.Fab)
+      (effects (font (size 1 1) (thickness 0.15)))
+    )
+    (fp_text user %R (at 0.3 0) (layer F.Fab)
+      (effects (font (size 1 1) (thickness 0.15)))
+    )
+    (fp_circle (center 0 0) (end 3.5 0) (layer Cmts.User) (width 0.15))
+    (fp_circle (center 0 0) (end 3.75 0) (layer F.CrtYd) (width 0.05))
+    (pad 1 np_thru_hole circle (at 0 0) (size 3.5 3.5) (drill 3.5) (layers *.Cu *.Mask))
+  )
   (gr_line (start 75 140) (end 75 50) (layer Eco1.User) (width 0.2))
   (gr_line (start 225 140) (end 227.5 140) (layer Eco1.User) (width 0.2))
@@
   (gr_line (start 230 145) (end 70 145) (layer Edge.Cuts) (width 0.15))
   (gr_line (start 230 45) (end 230 145) (layer Edge.Cuts) (width 0.15))
+  (via (at 77.5 137.5) (size 3.5) (drill 3) (layers F.Cu B.Cu) (net 0))
 )

Commit message: routed
Parts:
- removed the REF** at (219.0, 139.0)
- removed the REF** at (219.0, 50.0)
- added REF**: MountingHole_3.5mm, Mounting_Holes:MountingHole_3.5mm, F.Cu at (218.8, 50.0)
- added REF**: MountingHole_3.5mm, Mounting_Holes:MountingHole_3.5mm, F.Cu at (218.8, 140.0)
- J3, J4, J5: footprint Connectors:Pin_d0.7mm_L6.5mm_W1.8mm_FlatFork -> Flachsteceker:216843-1
- moved J5 26.8 mm to (123.0, 55.5), turned to 0 degrees
- moved J3 6.99 mm to (149.0, 55.5)
- moved J2 3.00 mm to (185.0, 122.0)
- moved J4 1.69 mm to (149.0, 133.5), turned to 180 degrees
- moved RV1 0.48 mm to (152.7, 96.5)
- moved F1 0.20 mm to (162.5, 136.4)
Connections:
- net Net-(C8-Pad1) renamed /HC_OUT
- net Net-(Q14-Pad1) renamed /HC_Q16_C
- net Net-(Q14-Pad2) renamed /HC_Q14_C
- net Net-(Q15-Pad1) renamed /HC_Q17_C
- net Net-(Q15-Pad2) renamed /HC_Q15_E
Routing:
- net /VSS_FUSED: track 0.00 -> 165.6 mm
- net /VCC_FUSED: track 0.00 -> 158.7 mm
- net Net-(C10-Pad2): track 0.00 -> 131.2 mm
- net /HC_OUT: track 0.00 -> 116.9 mm
- net Net-(Q10-Pad3): track 0.00 -> 103.0 mm
- net /HC_Q17_C: track 0.00 -> 90.7 mm
- net Net-(Q10-Pad2): track 0.00 -> 88.4 mm
- net /HC_Q14_C: track 0.00 -> 88.0 mm
- net /HC_Q16_C: track 0.00 -> 86.8 mm
- net Net-(D3-Pad1): track 0.00 -> 83.9 mm
- net Net-(D2-Pad2): track 0.00 -> 79.8 mm
- net /HC_Q15_E: track 0.00 -> 75.5 mm
- net Net-(C7-Pad2): track 0.00 -> 71.2 mm
- net Net-(C5-Pad2): track 0.00 -> 45.6 mm
- net Net-(Q5-Pad2): track 0.00 -> 43.3 mm
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- added copper zone on B.Cu, net GND
- added copper zone on F.Cu, net GND
Other:
- net class Default: trace_width 0.25 -> 0.5
- net class HIGH_CURRENT: trace_width 1 -> 2.1

Commit message: silkscreen
Routing:
- net Net-(Q12-Pad2): track 22.7 -> 27.5 mm
- net Net-(Q5-Pad2): track 43.3 -> 46.0 mm
- net Net-(C7-Pad2): track 71.2 -> 73.3 mm
- net Net-(C5-Pad2): track 45.6 -> 47.5 mm
- net Net-(C8-Pad2): track 13.8 -> 15.7 mm
- net /HC_Q15_E: track 75.5 -> 73.8 mm
- net Net-(Q2-Pad2): track 17.4 -> 19.1 mm
- net Net-(Q7-Pad2): track 6.77 -> 8.33 mm
- net /HC_Q16_C: track 86.8 -> 88.0 mm
- net Net-(Q11-Pad1): track 24.3 -> 25.5 mm
- net Net-(C10-Pad2): track 131.2 -> 132.4 mm
- net Net-(Q1-Pad1): track 12.5 -> 13.6 mm
- net Net-(Q11-Pad3): track 14.0 -> 14.9 mm
- net Net-(C6-Pad1): track 33.8 -> 34.3 mm
- net Net-(D3-Pad1): vias 0 -> 4
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Other:
- board text added: "+VCC"
- board text added: "-VCC"
- board text added: "80W HiFi Audio Amplifier"
- board text added: "BIAS+"
- board text added: "GND"
- board text added: "IC"
- board text added: "Ics"
- board text added: "Input"
- board text added: "Output"
- board text added: "Pero 01/2019"
- board text added: "VA/BIAS-"
- board text added: "VFB"
- board text added: "www.helentronica.com"

Commit message: in/out connectors, silkscreen check
Parts:
- removed the REF** at (80.0, 55.0)
- removed the REF** at (80.0, 135.0)
- removed the REF** at (218.8, 50.0)
- removed the REF** at (218.8, 140.0)
- added J6: Conn_01x01, Flachsteceker:216843-1, F.Cu at (83.0, 112.5)
- added J7: Conn_01x01, Flachsteceker:216843-1, F.Cu at (172.0, 122.3)
- added J8: Conn_01x01, Flachsteceker:216843-1, F.Cu at (123.0, 139.0)
- added REF**: MountingHole_3.5mm, Mounting_Holes:MountingHole_3.5mm, F.Cu at (87.0, 60.0)
- added REF**: MountingHole_3.5mm, Mounting_Holes:MountingHole_3.5mm, F.Cu at (90.0, 130.0)
- added REF**: MountingHole_3.5mm, Mounting_Holes:MountingHole_3.5mm, F.Cu at (217.5, 140.0)
- added REF**: MountingHole_3.5mm, Mounting_Holes:MountingHole_3.5mm, F.Cu at (219.0, 52.0)
- J1, J2: footprint Connectors:Pin_d0.7mm_L6.5mm_W1.8mm_FlatFork -> Flachsteceker:216843-1
- moved J1 15.7 mm to (83.0, 69.0)
- moved J2 14.1 mm to (172.0, 116.5)
Connections:
- net /HC_OUT renamed Net-(C8-Pad1)
- net /HC_Q14_C renamed Net-(Q14-Pad2)
- net /HC_Q15_E renamed Net-(Q15-Pad2)
- net /HC_Q16_C renamed Net-(Q14-Pad1)
- net /HC_Q17_C renamed Net-(Q15-Pad1)
Routing:
- net OUT: track 31.4 -> 46.9 mm
- net IN: track 7.15 -> 16.1 mm
- net Net-(C5-Pad2): track 47.5 -> 45.4 mm
- net Net-(D3-Pad1): vias 4 -> 0
- net GND: vias 114 -> 122
Other:
- board text added: "PWR GND"
- board text added: "SIG GND"
- board text removed: "GND"
