File: AudioAmp.kicad_pcb (KiCad board)
At the start: 2 copper layers, 160 x 100 mm, 84 parts, among them J1 Conn_01x01, J2 Conn_01x01, J3 Conn_01x01, J4 Conn_01x01, J5 Conn_01x01, J6 Conn_01x01, J7 Conn_01x01, J8 Conn_01x01, Q1 2N5401, Q10 2SD669, Q11 2SD669, Q12 2N5551, Q13 2N5401, Q14 2SD669, Q15 2SB649, Q16 2SA1302, Q17 2SC3281, Q2 2N5551, Q3 2N5401, Q4 2N5551, Q5 2N5401, Q6 2N5401, Q7 2N5551, Q8 2SD669, Q9 2SB649

Commit message: fixed Q9 and simulation
Connections:
- Q9 pad 1: Net-(C10-Pad1) -> Net-(Q9-Pad1)
- Q9 pad 2: Net-(Q9-Pad2) -> Net-(C10-Pad1)
- R14 pad 1: Net-(Q9-Pad2) -> Net-(Q9-Pad1)
- R20 pad 2: Net-(Q9-Pad2) -> Net-(Q9-Pad1)
Routing:
- net Net-(Q9-Pad2): track 21.9 -> 0.00 mm
- net Net-(Q9-Pad1): track 0.00 -> 16.1 mm
- net Net-(C10-Pad1): track 30.6 -> 34.2 mm

Commit message: fixed libraries, now works everything, including 3d models
Parts:
- C1, C2, C5, C6: footprint Capacitors_THT:CP_Radial_D10.0mm_P5.00mm -> Capacitor_THT:CP_Radial_D10.0mm_P5.00mm
- C11, C12, C13: footprint Capacitors_THT:C_Rect_L10.0mm_W4.0mm_P7.50mm_MKS4 -> Capacitor_THT:C_Rect_L10.0mm_W4.0mm_P7.50mm_MKS4
- C3, C4: footprint Capacitors_THT:CP_Radial_D22.0mm_P10.00mm_SnapIn -> Capacitor_THT:CP_Radial_D22.0mm_P10.00mm_SnapIn
- C7, C9: footprint Capacitors_THT:C_Rect_L10.0mm_W3.0mm_P7.50mm_MKS4 -> Capacitor_THT:C_Rect_L10.0mm_W3.0mm_P7.50mm_MKS4
- C8: footprint Capacitors_THT:C_Disc_D6.0mm_W2.5mm_P5.00mm -> Capacitor_THT:C_Disc_D6.0mm_W2.5mm_P5.00mm
- F1, F2: footprint Fuse_Holders_and_Fuses:Fuseholder5x20_horiz_open_inline_Type-I -> Fuse:Fuseholder_Cylinder-5x20mm_Schurter_0031_8201_Horizontal_Open
- R1, R10, R11, R12, R13, R14, R15, R16, R17, R18, R19, R2, R20, R21, R22, R23, R24, R25, R26, R27, R28, R29, R3, R30, R31, R32, R4, R5, R6, R7, R8, R9: footprint Resistors_THT:R_Axial_DIN0207_L6.3mm_D2.5mm_P10.16mm_Horizontal -> Resistor_THT:R_Axial_DIN0207_L6.3mm_D2.5mm_P10.16mm_Horizontal
- R35, R36: footprint Resistors_THT:R_Axial_DIN0516_L15.5mm_D5.0mm_P30.48mm_Horizontal -> Resistor_THT:R_Axial_DIN0516_L15.5mm_D5.0mm_P30.48mm_Horizontal
- RV1: footprint Potentiometers:Potentiometer_Trimmer_Piher_PT-10v10_Horizontal_Px10.0mm_Py5.0mm -> Potentiometer_THT:Potentiometer_Piher_PT-10-V10_Vertical
