File: Preamp/Preamp.kicad_pcb (KiCad board)
At the start: 2 copper layers, 83 x 54 mm, 55 parts, among them J1 +20, J10 R Out+, J11 R Out-, J2 GND, J3 -20, J4 L In+, J5 L In-, J6 R In+, J7 R In-, J8 L Out+, J9 L Out-, U1 L7815, U2 L7915, U3 OPA2134, U4 OPA2134

Commit message: silkscreen, preorder ready
Parts:
- moved J9 1.38 mm to (162.8, 76.2)
- moved J8 0.83 mm to (168.2, 76.3)
- moved J11 0.42 mm to (173.6, 76.3)
Connections:
- J11 pad 1: Net-(J11-Pad1) -> GND
Routing:
- net +15V: track 65.1 -> 79.0 mm
- net Net-(J11-Pad1): track 5.08 -> 0.00 mm
- net GND: track 0.00 -> 5.08 mm
- net Net-(C10-Pad1): track 30.5 -> 33.8 mm
- net Net-(R11-Pad1): track 109.5 -> 112.0 mm
- net Net-(C11-Pad1): track 46.1 -> 47.2 mm
Other:
- board text added: "7fda80a"
- board text added: "L In+"
- board text added: "L In-"
- board text added: "L Out+"
- board text added: "L Out-"
- board text added: "R In+"
- board text added: "R In-"
- board text added: "R Out+"
- board text added: "R Out-"

Commit message: ordered
Other:
- board text added: "2e9ee12"
- board text removed: "7fda80a"
Changed lines of the file:
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@@
     (34 B.Paste user hide)
     (35 F.Paste user hide)
-    (36 B.SilkS user hide)
-    (37 F.SilkS user)
+    (36 B.SilkS user)
+    (37 F.SilkS user hide)
     (38 B.Mask user hide)
     (39 F.Mask user hide)
@@
     (47 F.CrtYd user hide)
     (48 B.Fab user hide)
-    (49 F.Fab user hide)
+    (49 F.Fab user)
   )
   (setup
@@
     (visible_elements 7FFFFFFF)
     (pcbplotparams
-      (layerselection 0x010fc_ffffffff)
+      (layerselection 0x010f0_ffffffff)
       (usegerberextensions false)
       (usegerberattributes false)
@@
       (psa4output false)
       (plotreference true)
-      (plotvalue true)
+      (plotvalue false)
       (plotinvisibletext false)
       (padsonsilk false)
@@
       (outputformat 1)
       (mirror false)
-      (drillshape 1)
+      (drillshape 0)
       (scaleselection 1)
-      (outputdirectory ""))
+      (outputdirectory "./Gerbers"))
   )
   (net 0 "")
@@
     (effects (font (size 1.5 1.2) (thickness 0.2)))
   )
-  (gr_text 7fda80a (at 185 83 270) (layer B.SilkS)
+  (gr_text 2e9ee12 (at 185 83 270) (layer B.SilkS)
     (effects (font (size 2.5 2) (thickness 0.3)) (justify mirror))
   )
