File: Preamp/Preamp.sch (KiCad schematic (older format))
At the start: 23 parts

Commit message: preamp footprints
Parts:
- removed R?: R, symbol Device:R
- removed RV? (x2): 100k, symbol Device:R_POT
- added C1, C2: 10u, symbol Device:CP
- added C10, C11, C12, C13, C14, C7, C8, C9: 1u, symbol Device:C
- added C5, C6: 100n, symbol Device:C
- added J1: +20, Connectors:Pin_d1.0mm_L10.0mm, symbol Connector_Generic:Conn_01x01
- added J10: R Out+, Flachsteceker:216843-1, symbol Connector_Generic:Conn_01x01
- added J11: R Out-, Flachsteceker:216843-1, symbol Connector_Generic:Conn_01x01
- added J2: GND, Connectors:Pin_d1.0mm_L10.0mm, symbol Connector_Generic:Conn_01x01
- added J3: -20, Connectors:Pin_d1.0mm_L10.0mm, symbol Connector_Generic:Conn_01x01
- added J4: L In+, Connectors:Pin_d1.0mm_L10.0mm, symbol Connector_Generic:Conn_01x01
- added J5: L In-, Connectors:Pin_d1.0mm_L10.0mm, symbol Connector_Generic:Conn_01x01
- added J6: R In+, Connectors:Pin_d1.0mm_L10.0mm, symbol Connector_Generic:Conn_01x01
- added J7: R In-, Connectors:Pin_d1.0mm_L10.0mm, symbol Connector_Generic:Conn_01x01
- added J8: L Out+, Flachsteceker:216843-1, symbol Connector_Generic:Conn_01x01
- added J9: L Out-, Flachsteceker:216843-1, symbol Connector_Generic:Conn_01x01
- added R11: 100k, Potentiometers:Potentiometer_Piher_PC-16_Double_Vertical, symbol Pero_Kicad_Libraray:R_POT_x2
- added R13: 15k, Resistors_THT:R_Axial_DIN0207_L6.3mm_D2.5mm_P10.16mm_Horizontal, symbol Device:R
- added R15, R17: 10k, Resistors_THT:R_Axial_DIN0207_L6.3mm_D2.5mm_P10.16mm_Horizontal, symbol Device:R
- added R18, R19: 100R, Resistors_THT:R_Axial_DIN0207_L6.3mm_D2.5mm_P10.16mm_Horizontal, symbol Device:R
- added R20, R21: 100k, Resistors_THT:R_Axial_DIN0207_L6.3mm_D2.5mm_P10.16mm_Horizontal, symbol Device:R
- added U1: L7815, TO_SOT_Packages_THT:TO-220-3_Vertical, symbol Regulator_Linear:L7815
- added U2: L7915, TO_SOT_Packages_THT:TO-220-3_Vertical, symbol Regulator_Linear:L7915
- added unit 2 of U4
- added unit 3 of U4
- R1, R10, R14, R16, R2, R3, R4, R5, R6, R7, R8, R9: renamed from R?; footprint (none) -> Resistors_THT:R_Axial_DIN0207_L6.3mm_D2.5mm_P10.16mm_Horizontal
- R12: renamed from R?; value R -> 15k; footprint (none) -> Resistors_THT:R_Axial_DIN0207_L6.3mm_D2.5mm_P10.16mm_Horizontal
- U3, U4: renamed from U?; footprint (none) -> Housings_SOIC:SO-8_5.3x6.2mm_Pitch1.27mm
- gave numbers to parts that had none: 3
Connections:
- net GND: now also R12.2, R14.2, RV1.2, C1.2, C13.1, C14.1, C2.1, C5.2, C6.1, C7.1, C8.1, J2.1 (Pin_1), J5.1 (Pin_1), J7.1 (Pin_1), J9.1 (Pin_1), R11.3, R11.6, R13.2, R15.2, R20.2, R21.2, U1.2 (GND), U2.1 (GND)
- net L_in: now also J4.1 (Pin_1)
- net R_in: now also J6.1 (Pin_1)
- net at R12.1, U3.5 (+): now also R11.2
- net at R16.1, U3.7: now also R18.2
- net -15V: now reaches U3.4 (V-)
- net -15V: now also C14.2, C6.2, C8.2, U2.3 (VO), U4.4 (V-)
- net +15V: now reaches U3.8 (V+)
- net +15V: now also C13.2, C5.1, C7.2, U1.3 (OUT), U4.8 (V+)
- net at R9.1, RV1.1: now also R11.1
- net at R10.1, RV1.3: now also R11.4
- new net: R11.5, R13.1, U4.5 (+)
- new net: C10.2, C9.2, R18.1
- new net: C10.1, C9.1, J8.1 (Pin_1), R20.1
- new net: R15.1, R17.2, U4.6 (-)
- new net: R17.1, R19.2, U4.7
- new net: C11.2, C12.2, R19.1
- new net: C11.1, C12.1, J10.1 (Pin_1), R21.1
- new net: C1.1, J1.1 (Pin_1), U1.1 (IN)
- new net: C2.2, J3.1 (Pin_1), U2.2 (VI)
Other:
- moved on the sheet: R14, R16, RV1, U3C

Commit message: routing finished
Parts:
- C1, C2: footprint (none) -> Capacitors_THT:CP_Radial_Tantal_D5.0mm_P5.00mm
- C10, C11, C12, C3, C4, C9: footprint (none) -> Capacitors_THT:C_Rect_L10.3mm_W5.0mm_P7.50mm_MKS4
- C13, C14, C7, C8: footprint (none) -> Capacitors_THT:C_Disc_D5.1mm_W3.2mm_P5.00mm
- C5, C6: footprint (none) -> Capacitors_THT:C_Rect_L10.0mm_W2.5mm_P7.50mm_MKS4
- RV1: footprint (none) -> Potentiometers:Potentiometer_Trimmer_Piher_PT-10h2.5_Vertical_Px2.5mm_Py5.0mm
- U3, U4: footprint Housings_SOIC:SO-8_5.3x6.2mm_Pitch1.27mm -> Housings_DIP:DIP-8_W7.62mm
Other:
- note added: "Stage 1: 6dB gain"
- note added: "Stage 2: 6dB gain"
Changed lines of the file:
@@
 F 0 "U3" H 4150 3267 50  0000 C CNN
 F 1 "OPA2134" H 4150 3176 50  0000 C CNN
-F 2 "Housings_SOIC:SO-8_5.3x6.2mm_Pitch1.27mm" H 4150 2900 50  0001 C CNN
+F 2 "Housings_DIP:DIP-8_W7.62mm" H 4150 2900 50  0001 C CNN
 F 3 "http://www.ti.com/lit/ds/symlink/opa134.pdf" H 4150 2900 50  0001 C CNN
 	1    4150 2900
@@
 F 0 "U3" H 8050 3367 50  0000 C CNN
 F 1 "OPA2134" H 8050 3276 50  0000 C CNN
-F 2 "Housings_SOIC:SO-8_5.3x6.2mm_Pitch1.27mm" H 8050 3000 50  0001 C CNN
+F 2 "Housings_DIP:DIP-8_W7.62mm" H 8050 3000 50  0001 C CNN
 F 3 "http://www.ti.com/lit/ds/symlink/opa134.pdf" H 8050 3000 50  0001 C CNN
 	2    8050 3000
@@
 F 0 "U3" H 9058 1496 50  0000 L CNN
 F 1 "OPA2134" H 9058 1405 50  0000 L CNN
-F 2 "Housings_SOIC:SO-8_5.3x6.2mm_Pitch1.27mm" H 9100 1450 50  0001 C CNN
+F 2 "Housings_DIP:DIP-8_W7.62mm" H 9100 1450 50  0001 C CNN
 F 3 "http://www.ti.com/lit/ds/symlink/opa134.pdf" H 9100 1450 50  0001 C CNN
 	3    9100 1450
@@
 F 0 "C3" V 1948 2800 50  0000 C CNN
 F 1 "1u" V 2039 2800 50  0000 C CNN
-F 2 "" H 2200 2800 50  0001 C CNN
+F 2 "Capacitors_THT:C_Rect_L10.3mm_W5.0mm_P7.50mm_MKS4" H 2200 2800 50  0001 C CNN
 F 3 "" H 2200 2800 50  0001 C CNN
 	1    2200 2800
@@
 F 0 "RV1" H 5681 3696 50  0000 R CNN
 F 1 "10k" H 5681 3605 50  0000 R CNN
-F 2 "" H 5750 3650 50  0001 C CNN
+F 2 "Potentiometers:Potentiometer_Trimmer_Piher_PT-10h2.5_Vertical_Px2.5mm_Py5.0mm" H 5750 3650 50  0001 C CNN
 F 3 "" H 5750 3650 50  0001 C CNN
 	1    5750 3650
@@
 F 0 "U4" H 4150 4767 50  0000 C CNN
 F 1 "OPA2134" H 4150 4676 50  0000 C CNN
-F 2 "Housings_SOIC:SO-8_5.3x6.2mm_Pitch1.27mm" H 4150 4400 50  0001 C CNN
+F 2 "Housings_DIP:DIP-8_W7.62mm" H 4150 4400 50  0001 C CNN
 F 3 "http://www.ti.com/lit/ds/symlink/opa134.pdf" H 4150 4400 50  0001 C CNN
 	1    4150 4400
@@
 F 0 "C4" V 1948 4300 50  0000 C CNN
 F 1 "1u" V 2039 4300 50  0000 C CNN
-F 2 "" H 2200 4300 50  0001 C CNN
+F 2 "Capacitors_THT:C_Rect_L10.3mm_W5.0mm_P7.50mm_MKS4" H 2200 4300 50  0001 C CNN
 F 3 "" H 2200 4300 50  0001 C CNN
 	1    2200 4300
@@
 F 0 "C10" V 9200 3000 50  0000 C CNN
 F 1 "1u" V 9500 3000 50  0000 C CNN
-F 2 "" H 9350 3000 50  0001 C CNN
+F 2 "Capacitors_THT:C_Rect_L10.3mm_W5.0mm_P7.50mm_MKS4" H 9350 3000 50  0001 C CNN
 F 3 "" H 9350 3000 50  0001 C CNN
 	1    9350 3000
@@
 F 0 "C9" V 9200 2600 50  0000 C CNN
 F 1 "1u" V 9500 2600 50  0000 C CNN
-F 2 "" H 9350 2600 50  0001 C CNN
+F 2 "Capacitors_THT:C_Rect_L10.3mm_W5.0mm_P7.50mm_MKS4" H 9350 2600 50  0001 C CNN
 F 3 "" H 9350 2600 50  0001 C CNN
 	1    9350 2600
@@
 F 0 "U4" H 8050 4867 50  0000 C CNN
 F 1 "OPA2134" H 8050 4776 50  0000 C CNN
-F 2 "Housings_SOIC:SO-8_5.3x6.2mm_Pitch1.27mm" H 8050 4500 50  0001 C CNN
+F 2 "Housings_DIP:DIP-8_W7.62mm" H 8050 4500 50  0001 C CNN
 F 3 "http://www.ti.com/lit/ds/symlink/opa134.pdf" H 8050 4500 50  0001 C CNN
 	2    8050 4500
@@
 F 0 "C12" V 9200 4500 50  0000 C CNN
 F 1 "1u" V 9500 4500 50  0000 C CNN
-F 2 "" H 9350 4500 50  0001 C CNN
+F 2 "Capacitors_THT:C_Rect_L10.3mm_W5.0mm_P7.50mm_MKS4" H 9350 4500 50  0001 C CNN
 F 3 "" H 9350 4500 50  0001 C CNN
 	1    9350 4500
@@
 F 0 "C11" V 9200 4100 50  0000 C CNN
 F 1 "1u" V 9500 4100 50  0000 C CNN
-F 2 "" H 9350 4100 50  0001 C CNN
+F 2 "Capacitors_THT:C_Rect_L10.3mm_W5.0mm_P7.50mm_MKS4" H 9350 4100 50  0001 C CNN
 F 3 "" H 9350 4100 50  0001 C CNN
 	1    9350 4100
@@
 F 0 "C8" V 9150 1800 50  0000 C CNN
 F 1 "1u" V 9450 1800 50  0000 C CNN
-F 2 "" H 9300 1800 50  0001 C CNN
+F 2 "Capacitors_THT:C_Disc_D5.1mm_W3.2mm_P5.00mm" H 9300 1800 50  0001 C CNN
 F 3 "" H 9300 1800 50  0001 C CNN
 	1    9300 1800
@@
 F 0 "C7" V 9150 1100 50  0000 C CNN
 F 1 "1u" V 9450 1100 50  0000 C CNN
-F 2 "" H 9300 1100 50  0001 C CNN
+F 2 "Capacitors_THT:C_Disc_D5.1mm_W3.2mm_P5.00mm" H 9300 1100 50  0001 C CNN
 F 3 "" H 9300 1100 50  0001 C CNN
 	1    9300 1100
@@
 F 0 "U4" H 10258 1496 50  0000 L CNN
 F 1 "OPA2134" H 10258 1405 50  0000 L CNN
-F 2 "Housings_SOIC:SO-8_5.3x6.2mm_Pitch1.27mm" H 10300 1450 50  0001 C CNN
+F 2 "Housings_DIP:DIP-8_W7.62mm" H 10300 1450 50  0001 C CNN
 F 3 "http://www.ti.com/lit/ds/symlink/opa134.pdf" H 10300 1450 50  0001 C CNN
 	3    10300 1450
@@
 F 0 "C14" V 10350 1800 50  0000 C CNN
 F 1 "1u" V 10650 1800 50  0000 C CNN
-F 2 "" H 10500 1800 50  0001 C CNN
+F 2 "Capacitors_THT:C_Disc_D5.1mm_W3.2mm_P5.00mm" H 10500 1800 50  0001 C CNN
 F 3 "" H 10500 1800 50  0001 C CNN
 	1    10500 1800
@@
 F 0 "C13" V 10350 1100 50  0000 C CNN
 F 1 "1u" V 10650 1100 50  0000 C CNN
-F 2 "" H 10500 1100 50  0001 C CNN
+F 2 "Capacitors_THT:C_Disc_D5.1mm_W3.2mm_P5.00mm" H 10500 1100 50  0001 C CNN
 F 3 "" H 10500 1100 50  0001 C CNN
 	1    10500 1100
@@
 F 0 "C1" H 2268 1346 50  0000 L CNN
 F 1 "10u" H 2268 1255 50  0000 L CNN
-F 2 "" H 2188 1150 50  0001 C CNN
+F 2 "Capacitors_THT:CP_Radial_Tantal_D5.0mm_P5.00mm" H 2188 1150 50  0001 C CNN
 F 3 "~" H 2150 1300 50  0001 C CNN
 	1    2150 1300
@@
 F 0 "C2" H 2268 1746 50  0000 L CNN
 F 1 "10u" H 2268 1655 50  0000 L CNN
-F 2 "" H 2188 1550 50  0001 C CNN
+F 2 "Capacitors_THT:CP_Radial_Tantal_D5.0mm_P5.00mm" H 2188 1550 50  0001 C CNN
 F 3 "~" H 2150 1700 50  0001 C CNN
 	1    2150 1700
@@
 F 0 "C5" H 3215 1346 50  0000 L CNN
 F 1 "100n" H 3215 1255 50  0000 L CNN
-F 2 "" H 3138 1150 50  0001 C CNN
+F 2 "Capacitors_THT:C_Rect_L10.0mm_W2.5mm_P7.50mm_MKS4" H 3138 1150 50  0001 C CNN
 F 3 "~" H 3100 1300 50  0001 C CNN
 	1    3100 1300
@@
 F 0 "C6" H 3215 1746 50  0000 L CNN
 F 1 "100n" H 3215 1655 50  0000 L CNN
-F 2 "" H 3138 1550 50  0001 C CNN
+F 2 "Capacitors_THT:C_Rect_L10.0mm_W2.5mm_P7.50mm_MKS4" H 3138 1550 50  0001 C CNN
 F 3 "~" H 3100 1700 50  0001 C CNN
 	1    3100 1700
@@
 	1    0    0    1
 $EndComp
+Text Notes 3700 2350 0    50   ~ 0
+Stage 1: 6dB gain
+Text Notes 7650 2350 0    50   ~ 0
+Stage 2: 6dB gain
 $EndSCHEMATC

Commit message: silkscreen, preorder ready
Connections:
- net GND: now also J11.1 (Pin_1)
Changed lines of the file:
@@
 Connection ~ 9700 4500
 Wire Wire Line
-	9700 5000 9700 5150
+	9700 5000 9700 5100
 $Comp
 L power:GND #PWR0104
@@
 	1    0    0    1
 $EndComp
-Wire Wire Line
-	10200 5100 9700 5100
 $Comp
 L Connector_Generic:Conn_01x01 J1
@@
 Text Notes 7650 2350 0    50   ~ 0
 Stage 2: 6dB gain
+Wire Wire Line
+	10200 5100 9700 5100
+Connection ~ 9700 5100
+Wire Wire Line
+	9700 5100 9700 5150
 $EndSCHEMATC

Commit message: fixed libraries, now works everything, including 3d models
Parts:
- C1: footprint Capacitors_THT:CP_Radial_Tantal_D5.0mm_P5.00mm -> Potentiometer_THT:Potentiometer_Piher_PT-10-H05_Horizontal
- C10, C11, C12, C3, C4, C9: footprint Capacitors_THT:C_Rect_L10.3mm_W5.0mm_P7.50mm_MKS4 -> Capacitor_THT:C_Rect_L10.3mm_W5.0mm_P7.50mm_MKS4
- C13, C14, C7, C8: footprint Capacitors_THT:C_Disc_D5.1mm_W3.2mm_P5.00mm -> Capacitor_THT:C_Disc_D5.1mm_W3.2mm_P5.00mm
- C2: footprint Capacitors_THT:CP_Radial_Tantal_D5.0mm_P5.00mm -> Capacitor_THT:CP_Radial_Tantal_D5.0mm_P5.00mm
- C5, C6: footprint Capacitors_THT:C_Rect_L10.0mm_W2.5mm_P7.50mm_MKS4 -> Capacitor_THT:C_Rect_L10.0mm_W2.5mm_P7.50mm_MKS4
- R1, R10, R12, R13, R14, R15, R16, R17, R18, R19, R2, R20, R21, R3, R4, R5, R6, R7, R8, R9: footprint Resistors_THT:R_Axial_DIN0207_L6.3mm_D2.5mm_P10.16mm_Horizontal -> Resistor_THT:R_Axial_DIN0207_L6.3mm_D2.5mm_P10.16mm_Horizontal
- R11: footprint Potentiometers:Potentiometer_Piher_PC-16_Double_Vertical -> Potentiometer_THT:Potentiometer_Piher_PC-16_Dual_Horizontal
- U1, U2: footprint TO_SOT_Packages_THT:TO-220-3_Vertical -> Package_TO_SOT_THT:TO-220-3_Vertical
- U3, U4: footprint Housings_DIP:DIP-8_W7.62mm -> Package_DIP:DIP-8_W7.62mm
