File: Power/Power.kicad_pcb (KiCad board)
At the start: 2 copper layers, 102.6 x 105.7 mm, 11 parts, among them J1 Trafo, J2 Power L, J3 Power R, J4 Power Preamp

Commit message: put actual mounting holes insted of vias in Power pcb
Parts:
- added REF**: MountingHole_3.5mm, MountingHole:MountingHole_3.5mm, F.Cu at (113.7, 153.7)
- added REF**: MountingHole_3.5mm, MountingHole:MountingHole_3.5mm, F.Cu at (205.7, 153.7)
- added REF**: MountingHole_3.5mm, MountingHole:MountingHole_3.5mm, F.Cu at (206.4, 57.8)
- added REF**: MountingHole_3.5mm, MountingHole:MountingHole_3.5mm, F.Cu at (113.7, 57.8)
Routing:
- net (no net): vias 4 -> 0
Changed lines of the file:
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@@
-(kicad_pcb (version 20171130) (host pcbnew "(5.1.2)-2")
+(kicad_pcb (version 20171130) (host pcbnew "(5.1.5)-3")
   (general
     (thickness 1.6)
     (drawings 11)
-    (tracks 55)
+    (tracks 51)
     (zones 0)
-    (modules 11)
+    (modules 15)
     (nets 6)
   )
@@
   )
   (layers
-    (0 F.Cu signal hide)
+    (0 F.Cu signal)
     (31 B.Cu signal hide)
     (32 B.Adhes user hide)
@@
   )
   (setup
-    (last_trace_width 2)
+    (last_trace_width 0.25)
     (user_trace_width 0.25)
     (user_trace_width 0.5)
@@
     (mod_text_size 1 1)
     (mod_text_width 0.15)
-    (pad_size 1.524 1.524)
-    (pad_drill 0.762)
+    (pad_size 3.5 3.5)
+    (pad_drill 3.5)
     (pad_to_mask_clearance 0.051)
     (solder_mask_min_width 0.25)
@@
     (add_net +24V)
     (add_net -24V)
+  )
+  (module MountingHole:MountingHole_3.5mm (layer F.Cu)
+    (at 113.665 153.67)
+    (descr "Mounting Hole 3.5mm, no annular")
+    (tags "mounting hole 3.5mm no annular")
+    (attr virtual)
+    (fp_text reference REF** (at 0 -4.5) (layer F.SilkS)
+      (effects (font (size 1 1) (thickness 0.15)))
+    )
+    (fp_text value MountingHole_3.5mm (at 0 4.5) (layer F.Fab)
+      (effects (font (size 1 1) (thickness 0.15)))
+    )
+    (fp_text user %R (at 0.3 0) (layer F.Fab)
+      (effects (font (size 1 1) (thickness 0.15)))
+    )
+    (fp_circle (center 0 0) (end 3.5 0) (layer Cmts.User) (width 0.15))
+    (fp_circle (center 0 0) (end 3.75 0) (layer F.CrtYd) (width 0.05))
+    (pad "" np_thru_hole circle (at -5.665 0.33) (size 3.5 3.5) (drill 3.5) (layers *.Cu *.Mask))
+  )
+  (module MountingHole:MountingHole_3.5mm (layer F.Cu)
+    (at 205.74 153.67)
+    (descr "Mounting Hole 3.5mm, no annular")
+    (tags "mounting hole 3.5mm no annular")
+    (attr virtual)
+    (fp_text reference REF** (at 0 -4.5) (layer F.SilkS)
+      (effects (font (size 1 1) (thickness 0.15)))
+    )
+    (fp_text value MountingHole_3.5mm (at 0 4.5) (layer F.Fab)
+      (effects (font (size 1 1) (thickness 0.15)))
+    )
+    (fp_text user %R (at 0.3 0) (layer F.Fab)
+      (effects (font (size 1 1) (thickness 0.15)))
+    )
+    (fp_circle (center 0 0) (end 3.5 0) (layer Cmts.User) (width 0.15))
+    (fp_circle (center 0 0) (end 3.75 0) (layer F.CrtYd) (width 0.05))
+    (pad "" np_thru_hole circle (at -5.74 0.33) (size 3.5 3.5) (drill 3.5) (layers *.Cu *.Mask))
+  )
+  (module MountingHole:MountingHole_3.5mm (layer F.Cu)
+    (at 206.375 57.785)
+    (descr "Mounting Hole 3.5mm, no annular")
+    (tags "mounting hole 3.5mm no annular")
+    (attr virtual)
+    (fp_text reference REF** (at 0 -4.5) (layer F.SilkS)
+      (effects (font (size 1 1) (thickness 0.15)))
+    )
+    (fp_text value MountingHole_3.5mm (at 0 4.5) (layer F.Fab)
+      (effects (font (size 1 1) (thickness 0.15)))
+    )
+    (fp_text user %R (at 0.3 0) (layer F.Fab)
+      (effects (font (size 1 1) (thickness 0.15)))
+    )
+    (fp_circle (center 0 0) (end 3.5 0) (layer Cmts.User) (width 0.15))
+    (fp_circle (center 0 0) (end 3.75 0) (layer F.CrtYd) (width 0.05))
+    (pad "" np_thru_hole circle (at -6.375 0.215) (size 3.5 3.5) (drill 3.5) (layers *.Cu *.Mask))
+  )
+  (module MountingHole:MountingHole_3.5mm (layer F.Cu)
+    (at 113.665 57.785)
+    (descr "Mounting Hole 3.5mm, no annular")
+    (tags "mounting hole 3.5mm no annular")
+    (attr virtual)
+    (fp_text reference REF** (at 0 -4.5) (layer F.SilkS)
+      (effects (font (size 1 1) (thickness 0.15)))
+    )
+    (fp_text value MountingHole_3.5mm (at 0 4.5) (layer F.Fab)
+      (effects (font (size 1 1) (thickness 0.15)))
+    )
+    (fp_circle (center 0 0) (end 3.75 0) (layer F.CrtYd) (width 0.05))
+    (fp_circle (center 0 0) (end 3.5 0) (layer Cmts.User) (width 0.15))
+    (fp_text user %R (at 0.3 0) (layer F.Fab)
+      (effects (font (size 1 1) (thickness 0.15)))
+    )
+    (pad "" np_thru_hole circle (at -5.665 0.215) (size 3.5 3.5) (drill 3.5) (layers *.Cu *.Mask))
   )
   (module AudioAmp:B43511-B9108-M (layer F.Cu)
@@
   (segment (start 196.088 76.312) (end 191.658 76.312) (width 2) (layer F.Cu) (net 1))
   (segment (start 191.658 76.312) (end 188.976 78.994) (width 2) (layer F.Cu) (net 1))
-  (via (at 108 58) (size 3.5) (drill 3) (layers F.Cu B.Cu) (net 0))
-  (via (at 200 58) (size 3.5) (drill 3) (layers F.Cu B.Cu) (net 0))
-  (via (at 108 154) (size 3.5) (drill 3) (layers F.Cu B.Cu) (net 0))
-  (via (at 200 154) (size 3.5) (drill 3) (layers F.Cu B.Cu) (net 0))
   (segment (start 121.158 113.792) (end 121.158 133.858) (width 2) (layer F.Cu) (net 3) (status 400000))
   (segment (start 133.662 146.362) (end 150.368 146.362) (width 2) (layer F.Cu) (net 3) (status 800000))
